File: BLDC_Motor_Driver/power.kicad_sch (KiCad schematic)
At the start: 12 parts, among them J701 Conn_01x02, U701 LM5164DDA

Commit message: finished power circuitry
Parts:
- added C204: 4.7uF, Capacitor_SMD:C_0603_1608Metric, symbol Device:C
- added C706: 1uF, Capacitor_SMD:C_0603_1608Metric, symbol Device:C
- added D203: RED LED, LED_SMD:LED_0603_1608Metric, symbol Device:LED
- added R207: 470, Resistor_SMD:R_0603_1608Metric, symbol Device:R_US
- added R705: 30k, Resistor_SMD:R_0603_1608Metric, symbol Device:R_US
- added R706: 10k, Resistor_SMD:R_0603_1608Metric, symbol Device:R_US
- added U204: TPS746-Q1, Package_SON:WSON-6-1EP_2x2mm_P0.65mm_EP1x1.6mm, symbol Regulator_Texas:TPS746-Q1
- added U702: TPS2116DRL, Package_TO_SOT_SMD:SOT-583-8, symbol Power_Management:TPS2116DRL
- J701: footprint (none) -> TerminalBlock_Phoenix:TerminalBlock_Phoenix_MKDS-1-2-3.81_1x02_P3.81mm_Horizontal
Connections:
- net 5V_OUT renamed 5V_REG
- net 5V_REG: now also R705.1, U702.3 (VIN1), U702.5 (MODE)
- net GND renamed EP
- net EP: now also C204.2, C706.2, D203.1 (K), R706.2, U204.3 (GND), U204.7 (EP), U702.1 (GND)
- new net: D203.2 (A), R207.2
- new net +3V3: C204.1, R207.1, U204.1 (OUT)
- new net 5V_COM: C706.1, U204.4 (EN), U204.6 (IN), U702.2 (VOUT), U702.7 (VOUT)
- new net PR1: R705.2, R706.1, U702.4 (PR1)
- new net USB_POWER: U702.6 (VIN2)
- no-connect marks 1 -> 3
Other:
- note added: "1.5-6.0V V_{IN} 1A Maximum Output"
- note added: "3V3 Regulator"
- note added: "Power Mux"
- note added: "TPS74633-Q1"
- company: (none) -> University of Illinois Urbana Champaign
- title: (none) -> BLDC Motor Inverter Power Circuitry

Commit message: hall effect done, adding testpoints/connectors
Other:
- note added: "Power Testpoints"
Changed lines of the file:
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@@
+	)
+	(rectangle
+		(start 92.71 68.58)
+		(end 125.73 111.76)
+		(stroke
+			(width 0)
+			(type dash)
+		)
+		(fill
+			(type none)
+		)
 	)
 	(rectangle
@@
 		)
 	)
+	(text "Power Testpoints"
+		(exclude_from_sim no)
+		(at 93.345 69.85 0)
+		(effects
+			(font
+				(size 2 2)
+				(thickness 0.4)
+				(bold yes)
+			)
+			(justify left top)
+		)
+	)
 	(junction
 		(at 219.71 34.29)
@@
 	(wire
 		(pts
+			(xy 104.14 95.25) (xy 104.14 92.71)
+		)
+		(stroke
+			(width 0)
+			(type default)
+		)
+	)
+	(wire
+		(pts
 			(xy 59.69 86.36) (xy 67.31 86.36)
 		)
@@
 	(wire
 		(pts
+			(xy 104.14 90.17) (xy 106.68 90.17)
+		)
+		(stroke
+			(width 0)
+			(type default)
+		)
+	)
+	(wire
+		(pts
 			(xy 88.9 54.61) (xy 88.9 53.34)
 		)
@@
 	(wire
 		(pts
+			(xy 106.68 92.71) (xy 104.14 92.71)
+		)
+		(stroke
+			(width 0)
+			(type default)
+		)
+	)
+	(wire
+		(pts
 			(xy 71.12 38.1) (xy 71.12 33.02)
 		)
@@
 	(wire
 		(pts
+			(xy 104.14 87.63) (xy 106.68 87.63)
+		)
+		(stroke
+			(width 0)
+			(type default)
+		)
+	)
+	(wire
+		(pts
 			(xy 58.42 43.18) (xy 58.42 44.45)
 		)
@@
 	(wire
 		(pts
+			(xy 104.14 85.09) (xy 104.14 83.82)
+		)
+		(stroke
+			(width 0)
+			(type default)
+		)
+	)
+	(wire
+		(pts
 			(xy 125.73 39.37) (xy 125.73 38.1)
 		)
@@
 		(pts
 			(xy 207.01 44.45) (xy 204.47 44.45)
+		)
+		(stroke
+			(width 0)
+			(type default)
+		)
+	)
+	(wire
+		(pts
+			(xy 106.68 85.09) (xy 104.14 85.09)
 		)
 		(stroke
@@
 			)
 			(justify right bottom)
+		)
+	)
+	(hierarchical_label "5V_COM"
+		(shape bidirectional)
+		(at 104.14 87.63 180)
+		(effects
+			(font
+				(size 1.27 1.27)
+			)
+			(justify right)
 		)
 	)
@@
 		)
 	)
+	(hierarchical_label "5V_REG"
+		(shape bidirectional)
+		(at 104.14 90.17 180)
+		(effects
+			(font
+				(size 1.27 1.27)
+			)
+			(justify right)
+		)
+	)
 	(hierarchical_label "USB_POWER"
 		(shape input)
@@
 	)
 	(symbol
+		(lib_id "power:GND")
+		(at 104.14 95.25 0)
+		(mirror y)
+		(unit 1)
+		(exclude_from_sim no)
+		(in_bom yes)
+		(on_board yes)
+		(dnp no)
+		(property "Reference" "#PWR0711"
+			(at 104.14 101.6 0)
+			(effects
+				(font
+					(size 1.27 1.27)
+				)
+				(hide yes)
+			)
+		)
+		(property "Value" "GND"
+			(at 104.14 100.33 0)
+			(effects
+				(font
+					(size 1.27 1.27)
+				)
+				(hide yes)
+			)
+		)
+		(property "Footprint" ""
+			(at 104.14 95.25 0)
+			(effects
+				(font
+					(size 1.27 1.27)
+				)
+				(hide yes)
+			)
+		)
+		(property "Datasheet" ""
+			(at 104.14 95.25 0)
+			(effects
+				(font
+					(size 1.27 1.27)
+				)
+				(hide yes)
+			)
+		)
+		(property "Description" "Power symbol creates a global label with name \"GND\" , ground"
+			(at 104.14 95.25 0)
+			(effects
+				(font
+					(size 1.27 1.27)
+				)
+				(hide yes)
+			)
+		)
+		(pin "1"
+		)
+		(instances
+			(project "BLDC_Motor_Driver"
+				(path "/f8816ca8-d12a-4d6e-83e4-586d8ea9408b/cc03d52c-49b6-4460-8b58-76a2106de344"
+					(reference "#PWR0711")
+					(unit 1)
+				)
+			)
+		)
+	)
+	(symbol
 		(lib_id "Device:C")
 		(at 58.42 39.37 0)
@@
 					(unit 1)
 				)
+			)
+		)
+	)
+	(symbol
+		(lib_id "power:+3V3")
+		(at 104.14 83.82 0)
+		(unit 1)
+		(exclude_from_sim no)
+		(in_bom yes)
+		(on_board yes)
+		(dnp no)
+		(fields_autoplaced yes)
+		(property "Reference" "#PWR0710"
+			(at 104.14 87.63 0)
+			(effects
+				(font
+					(size 1.27 1.27)
+				)
+				(hide yes)
+			)
+		)
+		(property "Value" "+3V3"
+			(at 104.14 78.74 0)
+			(effects
+				(font
+					(size 1.27 1.27)
+				)
+			)
+		)
+		(property "Footprint" ""
+			(at 104.14 83.82 0)
+			(effects
+				(font
+					(size 1.27 1.27)
+				)
+				(hide yes)
+			)
+		)
+		(property "Datasheet" ""
+			(at 104.14 83.82 0)
+			(effects
+				(font
+					(size 1.27 1.27)
+				)
+				(hide yes)
+			)
+		)
+		(property "Description" "Power symbol creates a global label with name \"+3V3\""
+			(at 104.14 83.82 0)
+			(effects
+				(font
+					(size 1.27 1.27)
+				)
+				(hide yes)
+			)
+		)
+		(pin "1"
+		)
+		(instances
+			(project "BLDC_Motor_Driver"
+				(path "/f8816ca8-d12a-4d6e-83e4-586d8ea9408b/cc03d52c-49b6-4460-8b58-76a2106de344"
+					(reference "#PWR0710")
+					(unit 1)
+				)

Commit message: new GateDriver subsheet. reorg connectors to root sheet
Parts:
- removed J701: Conn_01x02, TerminalBlock_Phoenix:TerminalBlock_Phoenix_MKDS-1-2-3.81_1x02_P3.81mm_Horizontal, symbol Connector_Generic:Conn_01x02
Connections:
- net +36V renamed 36V_VIN
- net +3V3 renamed 3.3V_REG
Other:
- note removed: "Power Input"
- note removed: "Power Testpoints"

Commit message: added breakout connector and reformatted some things
Connections:
- net 3.3V_REG renamed 3V3_REG
Changed lines of the file:
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@@
 		)
 	)
-	(hierarchical_label "3.3V_REG"
+	(hierarchical_label "3V3_REG"
 		(shape output)
 		(at 77.47 83.82 90)

Commit message: schematics more or less done
Parts:
- added C307, C308: 270uF, Capacitor_THT:CP_Radial_D16.0mm_P7.50mm, symbol Device:C
- added D302: SMBJ70A-13-F, Diode_SMD:D_SMB, symbol Diode:SM6T6V8A
- renumbered C701 to C301, C706 to C302, C204 to C303, C702 to C304, C703 to C305, C704 to C306, C705 to C309, D203 to D301, L701 to L301, R701 to R301, R207 to R302, R702 to R303, R703 to R304, R704 to R305, R705 to R306, R706 to R307, U204 to U301, U701 to U302, U702 to U303
Connections:
- net 36V_VIN: now also C307.1, C308.1, D302.1 (A1)
- net EP renamed GND
- net GND: now also C307.2, C308.2, D302.2 (A2)
Other:
- note added: "Bulk Capacitance"
- note added: "LM5164"
- note added: "TPS2116"
- company: University of Illinois Urbana Champaign -> University of Illinois Urbana-Champaign
- moved on the sheet: C301, C302, C303, C304, C305, C306, C309, D301, L301, R301, R302, R303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

Commit message: wired driver rst/status ios to mcu, layout setup
Parts:
- U302: footprint Package_SO:HSOP-8-1EP_3.9x4.9mm_P1.27mm_EP2.41x3.1mm_ThermalVias -> Package_SO:HSOP-8-1EP_3.9x4.9mm_P1.27mm_EP2.41x3.1mm
Changed lines of the file:
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@@
 			)
 		)
-		(property "Footprint" "Package_SO:HSOP-8-1EP_3.9x4.9mm_P1.27mm_EP2.41x3.1mm_ThermalVias"
+		(property "Footprint" "Package_SO:HSOP-8-1EP_3.9x4.9mm_P1.27mm_EP2.41x3.1mm"
 			(at 52.07 54.61 0)
 			(effects

Commit message: move elements to logical regions
Parts:
- U302: footprint Package_SO:HSOP-8-1EP_3.9x4.9mm_P1.27mm_EP2.41x3.1mm -> Package_SO:HSOP-8-1EP_3.9x4.9mm_P1.27mm_EP2.41x3.1mm_ThermalVias
Changed lines of the file:
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@@
 			)
 		)
-		(property "Datasheet" "https://www.digikey.com/en/products/detail/panasonic-electronic-components/EEU-FS2A271SB/9597113"
+		(property "Datasheet" "~"
 			(at 120.65 83.82 0)
 			(effects
@@
 			)
 		)
-		(property "Description" ""
+		(property "Description" "Resistor, US symbol"
 			(at 76.2 91.44 0)
 			(effects
@@
 			)
 		)
-		(property "Datasheet" "https://www.digikey.com/en/products/detail/diodes-incorporated/SMBJ70A-13-F/814628"
+		(property "Datasheet" "https://www.st.com/resource/en/datasheet/sm6t.pdf"
 			(at 132.08 82.55 0)
 			(effects
@@
 			)
 		)
-		(property "Description" "113V Clamp 5.3A Ipp Tvs Diode Surface Mount SMB"
+		(property "Description" "600W unidirectional Transil Transient Voltage Suppressor, 6.8Vrwm, DO-214AA"
 			(at 132.08 83.82 0)
 			(effects
@@
 	)
 	(symbol
+		(lib_id "power:PWR_FLAG")
+		(at 123.19 35.56 0)
+		(unit 1)
+		(exclude_from_sim no)
+		(in_bom yes)
+		(on_board yes)
+		(dnp no)
+		(fields_autoplaced yes)
+		(property "Reference" "#FLG01"
+			(at 123.19 33.655 0)
+			(effects
+				(font
+					(size 1.27 1.27)
+				)
+				(hide yes)
+			)
+		)
+		(property "Value" "PWR_FLAG"
+			(at 123.19 30.48 0)
+			(effects
+				(font
+					(size 1.27 1.27)
+				)
+			)
+		)
+		(property "Footprint" ""
+			(at 123.19 35.56 0)
+			(effects
+				(font
+					(size 1.27 1.27)
+				)
+				(hide yes)
+			)
+		)
+		(property "Datasheet" "~"
+			(at 123.19 35.56 0)
+			(effects
+				(font
+					(size 1.27 1.27)
+				)
+				(hide yes)
+			)
+		)
+		(property "Description" "Special symbol for telling ERC where power comes from"
+			(at 123.19 35.56 0)
+			(effects
+				(font
+					(size 1.27 1.27)
+				)
+				(hide yes)
+			)
+		)
+		(pin "1"
+		)
+		(instances
+			(project ""
+				(path "/f8816ca8-d12a-4d6e-83e4-586d8ea9408b/cc03d52c-49b6-4460-8b58-76a2106de344"
+					(reference "#FLG01")
+					(unit 1)
+				)
+			)
+		)
+	)
+	(symbol
 		(lib_id "Device:C")
 		(at 123.19 46.99 0)
@@
 			)
 		)
-		(property "Datasheet" "https://www.digikey.com/en/products/detail/panasonic-electronic-components/EEU-FS2A271SB/9597113"
+		(property "Datasheet" "~"
 			(at 107.95 83.82 0)
 			(effects
@@
 			)
 		)
-		(property "Footprint" "Package_SO:HSOP-8-1EP_3.9x4.9mm_P1.27mm_EP2.41x3.1mm"
+		(property "Footprint" "Package_SO:HSOP-8-1EP_3.9x4.9mm_P1.27mm_EP2.41x3.1mm_ThermalVias"
 			(at 52.07 54.61 0)
 			(effects
