File: BLDC_Motor_Driver/hbridge.kicad_sch (KiCad schematic)
At the start: 7 parts, among them Q1 CSD18540Q5B, Q2 CSD18540Q5B

Commit message: new GateDriver subsheet. reorg connectors to root sheet
Parts:
- renumbered C501 to C23, C203 to C24, C202 to C25, C201 to C26, Q1 to Q3, Q2 to Q4, R201 to R7

Commit message: schematics more or less done
Parts:
- renumbered C23 to C501, C24 to C502, C25 to C503, C26 to C504, Q3 to Q501, Q4 to Q502, R7 to R501
Other:
- company: (none) -> University of Illinois Urbana-Champaign
- title: (none) -> BLDC Motor Inverter H-Bridge Circuitry

Commit message: clean layout done. signoff required
Parts:
- added NT1: NetTie_2, NetTie:NetTie-2_THT_Pad0.3mm, symbol Device:NetTie_2
Connections:
- net GND: now also NT1.1
- new net CSN: NT1.2
Changed lines of the file:
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@@
+	)
+	(junction
+		(at 128.27 132.08)
+		(diameter 0)
+		(color 0 0 0 0)
 	)
 	(junction
@@
 	)
 	(junction
-		(at 128.27 132.08)
-		(diameter 0)
-		(color 0 0 0 0)
-	)
-	(junction
 		(at 149.86 90.17)
 		(diameter 0)
@@
 	(wire
 		(pts
+			(xy 134.62 132.08) (xy 135.89 132.08)
+		)
+		(stroke
+			(width 0)
+			(type default)
+		)
+	)
+	(wire
+		(pts
 			(xy 161.29 90.17) (xy 161.29 91.44)
 		)
@@
 	(wire
 		(pts
+			(xy 128.27 132.08) (xy 128.27 133.35)
+		)
+		(stroke
+			(width 0)
+			(type default)
+		)
+	)
+	(wire
+		(pts
 			(xy 128.27 104.14) (xy 149.86 104.14)
 		)
@@
 	(wire
 		(pts
+			(xy 128.27 132.08) (xy 129.54 132.08)
+		)
+		(stroke
+			(width 0)
+			(type default)
+		)
+	)
+	(wire
+		(pts
 			(xy 128.27 116.84) (xy 128.27 121.92)
 		)
@@
 	(wire
 		(pts
-			(xy 128.27 133.35) (xy 128.27 132.08)
+			(xy 128.27 130.81) (xy 128.27 132.08)
 		)
 		(stroke
@@
 	(wire
 		(pts
-			(xy 128.27 132.08) (xy 133.35 132.08)
-		)
-		(stroke
-			(width 0)
-			(type default)
-		)
-	)
-	(wire
-		(pts
 			(xy 149.86 104.14) (xy 149.86 105.41)
-		)
-		(stroke
-			(width 0)
-			(type default)
-		)
-	)
-	(wire
-		(pts
-			(xy 128.27 130.81) (xy 128.27 132.08)
 		)
 		(stroke
@@
 	(hierarchical_label "CSN"
 		(shape output)
-		(at 133.35 132.08 0)
+		(at 135.89 132.08 0)
 		(effects
 			(font
@@
 					(unit 1)
 				)
+			)
+		)
+	)
+	(symbol
+		(lib_id "Device:NetTie_2")
+		(at 132.08 132.08 0)
+		(unit 1)
+		(exclude_from_sim no)
+		(in_bom no)
+		(on_board yes)
+		(dnp no)
+		(fields_autoplaced yes)
+		(property "Reference" "NT1"
+			(at 132.08 127 0)
+			(effects
+				(font
+					(size 1.27 1.27)
+				)
+			)
+		)
+		(property "Value" "NetTie_2"
+			(at 132.08 129.54 0)
+			(effects
+				(font
+					(size 1.27 1.27)
+				)
+			)
+		)
+		(property "Footprint" "NetTie:NetTie-2_THT_Pad0.3mm"
+			(at 132.08 132.08 0)
+			(effects
+				(font
+					(size 1.27 1.27)
+				)
+				(hide yes)
+			)
+		)
+		(property "Datasheet" "~"
+			(at 132.08 132.08 0)
+			(effects
+				(font
+					(size 1.27 1.27)
+				)
+				(hide yes)
+			)
+		)
+		(property "Description" "Net tie, 2 pins"
+			(at 132.08 132.08 0)
+			(effects
+				(font
+					(size 1.27 1.27)
+				)
+				(hide yes)
+			)
+		)
+		(pin "2"
+		)
+		(pin "1"
+		)
+		(instances
+			(project ""
+				(path "/f8816ca8-d12a-4d6e-83e4-586d8ea9408b/9a7f02cf-afb2-4d66-9ae7-4e30a98b6980/4b4367ba-42d9-462c-bf20-675b6fbf5ab3"
+					(reference "NT1")
+					(unit 1)
+				)
+				(path "/f8816ca8-d12a-4d6e-83e4-586d8ea9408b/9a7f02cf-afb2-4d66-9ae7-4e30a98b6980/51dee69d-31d1-4b65-b804-890ce69bca2c"
+					(reference "NT3")
+					(unit 1)
+				)
+				(path "/f8816ca8-d12a-4d6e-83e4-586d8ea9408b/9a7f02cf-afb2-4d66-9ae7-4e30a98b6980/82226e03-7285-44d6-af19-d97077dd2091"
+					(reference "NT2")
+					(unit 1)
+				)
