File: Servo_Breakout/2bit_level_shifter.kicad_sch (KiCad schematic)
At the start: 3 parts, among them U401 TXS0102DCT

Commit message: servo board final cleanup
Parts:
- renumbered C401 to C301, C402 to C302, U401 to U301
Changed lines of the file:
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@@
 		(dnp no)
 		(fields_autoplaced yes)
-		(property "Reference" "C402"
+		(property "Reference" "C302"
 			(at 111.76 72.39 90)
 			(effects
@@
 			(project "Servo_Breakout"
 				(path "/d50da23a-d62e-4014-ae89-4f18c8c8c668/de7a4b00-096f-4422-b46a-78bd243039a7"
-					(reference "C402")
+					(reference "C302")
 					(unit 1)
 				)
@@
 		(dnp no)
 		(fields_autoplaced yes)
-		(property "Reference" "C401"
+		(property "Reference" "C301"
 			(at 96.52 72.39 90)
 			(effects
@@
 			(project ""
 				(path "/d50da23a-d62e-4014-ae89-4f18c8c8c668/de7a4b00-096f-4422-b46a-78bd243039a7"
-					(reference "C401")
+					(reference "C301")
 					(unit 1)
 				)
@@
 		(dnp no)
 		(fields_autoplaced yes)
-		(property "Reference" "U401"
+		(property "Reference" "U301"
 			(at 106.2833 113.03 0)
 			(effects
@@
 			(project ""
 				(path "/d50da23a-d62e-4014-ae89-4f18c8c8c668/de7a4b00-096f-4422-b46a-78bd243039a7"
-					(reference "U401")
+					(reference "U301")
 					(unit 1)
 				)

Commit message: servo breakout gerbers
Other:
- company: (none) -> University of Illinois Urbana-Champaign
- title: (none) -> Servo Breakout
Changed lines of the file:
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@@
 	(generator_version "9.0")
 	(paper "A4")
+	(title_block
+		(title "Servo Breakout")
+		(date "2026-03-24")
+		(rev "A")
+		(company "University of Illinois Urbana-Champaign")
+		(comment 4 "Contributors: Noah Breit, Thomas McManamen")
+	)
 	(junction
 		(at 101.6 80.01)
