File: Servo_Breakout/dc_buck.kicad_sch (KiCad schematic)
At the start: 19 parts, among them U301 STPS15H100CBY-TR, U302 BD9G500EFJ-LAE2

Commit message: servo board final cleanup
Parts:
- added R205: 0, Resistor_SMD:R_0805_2012Metric_Pad1.20x1.40mm_HandSolder, symbol Device:R_US
- C203: renamed from C303; value 15uF/100V -> 6800pF/50V; footprint Capacitor_SMD:C_2220_5750Metric_Pad1.97x5.40mm_HandSolder -> Capacitor_SMD:C_0805_2012Metric_Pad1.18x1.45mm_HandSolder
- renumbered C301 to C201, C302 to C202, C304 to C204, C305 to C205, C306 to C206, C307 to C207, C308 to C208, L301 to L201, R301 to R201, R302 to R202, R303 to R203, R304 to R204, R305 to R206, R306 to R207, R307 to R208, R308 to R209, U301 to U201, U302 to U202
Connections:
- net GND: now also R205.1; no longer C203.2, U202.3 (COMP)
- new net: C203.2, R205.2, U202.3 (COMP)
Other:
- note added: "Consider R204 = 5k for +6V Output (servo rated for 6.8V)"
- note added: "R205 in place of C1 in example application, leave open or short"
- note added: "VOUT = (R201 + R204 + R203) / (R203)"
- note removed: "Consider R304 = 5k for +6V Output (servo rated for 6.8V)"
Changed lines of the file:
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@@
 		)
 	)
-	(text "Consider R304 = 5k for +6V Output\n(servo rated for 6.8V)"
+	(text "Consider R204 = 5k for +6V Output\n(servo rated for 6.8V)"
 		(exclude_from_sim no)
 		(at 118.11 134.62 0)
@@
 		)
 	)
+	(text "R205 in place of C1 in example application, leave open or short"
+		(exclude_from_sim no)
+		(at 116.84 143.51 0)
+		(effects
+			(font
+				(size 1.27 1.27)
+			)
+		)
+	)
 	(text "VBUCK disabled when EN input is floating"
 		(exclude_from_sim no)
@@
 		)
 	)
-	(text "VOUT = (R301 + R304) / (R303)"
+	(text "VOUT = (R201 + R204 + R203) / (R203)"
 		(exclude_from_sim no)
 		(at 117.602 131.064 0)
@@
 	)
 	(junction
+		(at 119.38 100.33)
+		(diameter 0)
+		(color 0 0 0 0)
+	)
+	(junction
 		(at 82.55 90.17)
 		(diameter 0)
@@
 	)
 	(junction
-		(at 119.38 100.33)
-		(diameter 0)
-		(color 0 0 0 0)
-	)
-	(junction
 		(at 219.71 111.76)
 		(diameter 0)
@@
 	(wire
 		(pts
+			(xy 93.98 100.33) (xy 107.95 100.33)
+		)
+		(stroke
+			(width 0)
+			(type default)
+		)
+	)
+	(wire
+		(pts
 			(xy 134.62 68.58) (xy 134.62 95.25)
 		)
@@
 	(wire
 		(pts
+			(xy 115.57 100.33) (xy 119.38 100.33)
+		)
+		(stroke
+			(width 0)
+			(type default)
+		)
+	)
+	(wire
+		(pts
 			(xy 219.71 97.79) (xy 228.6 97.79)
 		)
@@
 		(pts
 			(xy 93.98 116.84) (xy 99.06 116.84)
-		)
-		(stroke
-			(width 0)
-			(type default)
-		)
-	)
-	(wire
-		(pts
-			(xy 93.98 100.33) (xy 119.38 100.33)
 		)
 		(stroke
@@
 		(dnp no)
 		(fields_autoplaced yes)
-		(property "Reference" "R307"
+		(property "Reference" "R208"
 			(at 182.88 111.7599 0)
 			(effects
@@
 			(project ""
 				(path "/d50da23a-d62e-4014-ae89-4f18c8c8c668/491641e7-7230-4c29-9234-fdc15d52c844"
-					(reference "R307")
+					(reference "R208")
 					(unit 1)
 				)
@@
 		(dnp no)
 		(fields_autoplaced yes)
-		(property "Reference" "C307"
+		(property "Reference" "C207"
 			(at 210.82 102.8699 0)
 			(effects
@@
 			(project "Servo_Breakout"
 				(path "/d50da23a-d62e-4014-ae89-4f18c8c8c668/491641e7-7230-4c29-9234-fdc15d52c844"
-					(reference "C307")
+					(reference "C207")
+					(unit 1)
+				)
+			)
+		)
+	)
+	(symbol
+		(lib_id "Device:R_US")
+		(at 111.76 100.33 90)
+		(unit 1)
+		(exclude_from_sim no)
+		(in_bom yes)
+		(on_board yes)
+		(dnp yes)
+		(property "Reference" "R205"
+			(at 111.76 95.25 90)
+			(effects
+				(font
+					(size 1.27 1.27)
+				)
+			)
+		)
+		(property "Value" "0"
+			(at 111.76 97.79 90)
+			(effects
+				(font
+					(size 1.27 1.27)
+				)
+			)
+		)
+		(property "Footprint" "Resistor_SMD:R_0805_2012Metric_Pad1.20x1.40mm_HandSolder"
+			(at 112.014 99.314 90)
+			(effects
+				(font
+					(size 1.27 1.27)
+				)
+				(hide yes)
+			)
+		)
+		(property "Datasheet" "~"
+			(at 111.76 100.33 0)
+			(effects
+				(font
+					(size 1.27 1.27)
+				)
+				(hide yes)
+			)
+		)
+		(property "Description" "Resistor, US symbol"
+			(at 111.76 100.33 0)
+			(effects
+				(font
+					(size 1.27 1.27)
+				)
+				(hide yes)
+			)
+		)
+		(pin "2"
+		)
+		(pin "1"
+		)
+		(instances
+			(project "Servo_Breakout"
+				(path "/d50da23a-d62e-4014-ae89-4f18c8c8c668/491641e7-7230-4c29-9234-fdc15d52c844"
+					(reference "R205")
 					(unit 1)
 				)
@@
 		(dnp no)
 		(fields_autoplaced yes)
-		(property "Reference" "R308"
+		(property "Reference" "R209"
 			(at 212.09 63.4999 0)
 			(effects
@@
 			(project ""
 				(path "/d50da23a-d62e-4014-ae89-4f18c8c8c668/491641e7-7230-4c29-9234-fdc15d52c844"
-					(reference "R308")
+					(reference "R209")
 					(unit 1)
 				)
@@
 		(dnp yes)
 		(fields_autoplaced yes)
-		(property "Reference" "R305"
+		(property "Reference" "R206"
 			(at 121.92 73.6599 0)
 			(effects
@@
 			(project ""
 				(path "/d50da23a-d62e-4014-ae89-4f18c8c8c668/491641e7-7230-4c29-9234-fdc15d52c844"
-					(reference "R305")
+					(reference "R206")
 					(unit 1)
 				)
@@
 		(on_board yes)
 		(dnp no)
-		(property "Reference" "C301"
+		(property "Reference" "C201"
 			(at 61.468 76.962 0)
 			(effects
@@
 			(project "Servo_Breakout"
 				(path "/d50da23a-d62e-4014-ae89-4f18c8c8c668/491641e7-7230-4c29-9234-fdc15d52c844"
-					(reference "C301")
+					(reference "C201")
 					(unit 1)
 				)
@@
 		(dnp no)
 		(fields_autoplaced yes)
-		(property "Reference" "U302"
+		(property "Reference" "U202"
 			(at 157.48 85.09 0)
 			(effects
@@
 			(project ""
 				(path "/d50da23a-d62e-4014-ae89-4f18c8c8c668/491641e7-7230-4c29-9234-fdc15d52c844"
-					(reference "U302")
+					(reference "U202")
 					(unit 1)
 				)
@@
 		(dnp no)
 		(fields_autoplaced yes)
-		(property "Reference" "L301"
+		(property "Reference" "L201"
 			(at 99.06 63.5 90)
 			(effects
@@
 			(project ""
 				(path "/d50da23a-d62e-4014-ae89-4f18c8c8c668/491641e7-7230-4c29-9234-fdc15d52c844"
-					(reference "L301")
+					(reference "L201")
 					(unit 1)
 				)
@@
 		(on_board yes)
 		(dnp no)
-		(property "Reference" "C303"
+		(property "Reference" "C203"
 			(at 115.57 110.998 90)
 			(effects
@@
 			)
 		)
-		(property "Value" "15uF/100V"
+		(property "Value" "6800pF/50V"
 			(at 115.57 113.792 90)
 			(effects
@@
 			)
 		)
-		(property "Footprint" "Capacitor_SMD:C_2220_5750Metric_Pad1.97x5.40mm_HandSolder"
+		(property "Footprint" "Capacitor_SMD:C_0805_2012Metric_Pad1.18x1.45mm_HandSolder"
 			(at 119.38 105.7148 0)
 			(effects
@@
 			(project ""
 				(path "/d50da23a-d62e-4014-ae89-4f18c8c8c668/491641e7-7230-4c29-9234-fdc15d52c844"
-					(reference "C303")
+					(reference "C203")
 					(unit 1)
 				)
@@
 		(dnp no)
 		(fields_autoplaced yes)
-		(property "Reference" "R303"
+		(property "Reference" "R203"
 			(at 102.87 110.49 90)
 			(effects
@@
 			(project "Servo_Breakout"
 				(path "/d50da23a-d62e-4014-ae89-4f18c8c8c668/491641e7-7230-4c29-9234-fdc15d52c844"
-					(reference "R303")
+					(reference "R203")
 					(unit 1)
 				)
@@
 		(dnp no)
 		(fields_autoplaced yes)
-		(property "Reference" "R306"
+		(property "Reference" "R207"
 			(at 161.29 62.23 90)
 			(effects
@@
 			(project ""
 				(path "/d50da23a-d62e-4014-ae89-4f18c8c8c668/491641e7-7230-4c29-9234-fdc15d52c844"
-					(reference "R306")
+					(reference "R207")
 					(unit 1)
 				)
@@
 		(on_board yes)
 		(dnp no)
-		(property "Reference" "R301"
+		(property "Reference" "R201"
 			(at 79.756 99.06 0)
 			(effects
@@
 			(project ""
 				(path "/d50da23a-d62e-4014-ae89-4f18c8c8c668/491641e7-7230-4c29-9234-fdc15d52c844"
-					(reference "R301")
+					(reference "R201")
 					(unit 1)
 				)
@@
 		(dnp no)
 		(fields_autoplaced yes)
-		(property "Reference" "R302"
+		(property "Reference" "R202"
 			(at 102.87 100.33 90)
 			(effects
@@
 			(project ""
 				(path "/d50da23a-d62e-4014-ae89-4f18c8c8c668/491641e7-7230-4c29-9234-fdc15d52c844"
-					(reference "R302")
+					(reference "R202")
 					(unit 1)
 				)
@@
 		(dnp no)
 		(fields_autoplaced yes)
-		(property "Reference" "C305"
+		(property "Reference" "C205"
 			(at 147.32 60.96 90)
 			(effects
@@
 			(project ""
 				(path "/d50da23a-d62e-4014-ae89-4f18c8c8c668/491641e7-7230-4c29-9234-fdc15d52c844"
-					(reference "C305")
+					(reference "C205")
 					(unit 1)
 				)
@@
 		(dnp no)
 		(fields_autoplaced yes)
-		(property "Reference" "U301"
+		(property "Reference" "U201"
 			(at 101.6 33.02 0)
 			(effects
@@
 			(project ""
 				(path "/d50da23a-d62e-4014-ae89-4f18c8c8c668/491641e7-7230-4c29-9234-fdc15d52c844"
-					(reference "U301")
+					(reference "U201")
 					(unit 1)
 				)
@@
 		(dnp no)
 		(fields_autoplaced yes)
-		(property "Reference" "C306"
+		(property "Reference" "C206"
 			(at 198.12 102.8699 0)
 			(effects
@@
 			(project ""
 				(path "/d50da23a-d62e-4014-ae89-4f18c8c8c668/491641e7-7230-4c29-9234-fdc15d52c844"
-					(reference "C306")
+					(reference "C206")
 					(unit 1)
 				)
@@
 		(dnp no)
 		(fields_autoplaced yes)
-		(property "Reference" "R304"
+		(property "Reference" "R204"
 			(at 110.49 120.65 90)
 			(effects
@@
 			(project "Servo_Breakout"
 				(path "/d50da23a-d62e-4014-ae89-4f18c8c8c668/491641e7-7230-4c29-9234-fdc15d52c844"
-					(reference "R304")
+					(reference "R204")
 					(unit 1)
 				)
@@
 		(dnp no)
 		(fields_autoplaced yes)
-		(property "Reference" "C308"
+		(property "Reference" "C208"
 			(at 223.52 102.8699 0)
 			(effects
@@
 			(project "Servo_Breakout"
 				(path "/d50da23a-d62e-4014-ae89-4f18c8c8c668/491641e7-7230-4c29-9234-fdc15d52c844"
-					(reference "C308")
+					(reference "C208")
 					(unit 1)
 				)
@@
 		(dnp yes)
 		(fields_autoplaced yes)
-		(property "Reference" "C304"
+		(property "Reference" "C204"
 			(at 123.19 83.8199 0)
 			(effects
@@
 			(project ""
 				(path "/d50da23a-d62e-4014-ae89-4f18c8c8c668/491641e7-7230-4c29-9234-fdc15d52c844"
-					(reference "C304")
+					(reference "C204")
 					(unit 1)
 				)
@@
 		(on_board yes)
 		(dnp no)
-		(property "Reference" "C302"
+		(property "Reference" "C202"
 			(at 75.438 76.708 0)
 			(effects
@@
 			(project ""
 				(path "/d50da23a-d62e-4014-ae89-4f18c8c8c668/491641e7-7230-4c29-9234-fdc15d52c844"
-					(reference "C302")
+					(reference "C202")
 					(unit 1)
 				)

Commit message: servo breakout gerbers
Other:
- company: (none) -> University of Illinois Urbana-Champaign
- title: 36V/5V 5A Buck -> Servo Breakout
Changed lines of the file:
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@@
 	(paper "A4")
 	(title_block
-		(title "36V/5V 5A Buck")
+		(title "Servo Breakout")
+		(date "2026-03-24")
+		(rev "A")
+		(company "University of Illinois Urbana-Champaign")
+		(comment 4 "Contributors: Noah Breit, Thomas McManamen")
 	)
 	(text "Snubbers"
